File: Eagle/PCM5102a_FG/PCM5102a_FG_Small_1.brd (EAGLE design)
At the start: 70.8 x 66 mm, 31 parts, among them IC1 PSOC_5LP_PROTOTIYPING_KIT, IC2 PCM5102A, IC3 TA48M033F, Q1 20MHz

Commit message: ハードウェア完成
Connections:
- removed net N$2: C4.2, C5.+
- net DGND: now also C4.2
- net N$1: now also C5.+
Routing:
- net N$2: track 12.7 -> 0.00 mm
- net N$1: track 2.54 -> 14.8 mm
- net DGND: track 245.9 -> 248.5 mm
Changed lines of the file:
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@@
 <layer number="41" name="tRestrict" color="4" fill="10" visible="yes" active="yes"/>
 <layer number="42" name="bRestrict" color="1" fill="10" visible="yes" active="yes"/>
-<layer number="43" name="vRestrict" color="2" fill="10" visible="yes" active="yes"/>
+<layer number="43" name="vRestrict" color="2" fill="10" visible="no" active="yes"/>
 <layer number="44" name="Drills" color="7" fill="1" visible="no" active="yes"/>
 <layer number="45" name="Holes" color="7" fill="1" visible="no" active="yes"/>
@@
 <contactref element="C3" pad="1"/>
 <contactref element="IC2" pad="16"/>
-<contactref element="C5" pad="-"/>
 <contactref element="IC2" pad="11"/>
 <contactref element="IC2" pad="12"/>
@@
 <wire x1="66.04" y1="12.7" x2="66.04" y2="25.4" width="0.4064" layer="16"/>
 <wire x1="66.04" y1="25.4" x2="66.04" y2="27.94" width="0.4064" layer="16"/>
-<wire x1="38.1" y1="22.86" x2="45.72" y2="22.86" width="0.4064" layer="16"/>
-<wire x1="45.72" y1="22.86" x2="45.72" y2="25.4" width="0.4064" layer="16"/>
 <wire x1="17.78" y1="12.7" x2="17.78" y2="22.86" width="0.4064" layer="16"/>
 <wire x1="17.78" y1="22.86" x2="25.4" y2="22.86" width="0.4064" layer="16"/>
-<wire x1="25.4" y1="22.86" x2="38.1" y2="22.86" width="0.4064" layer="16"/>
 <wire x1="22.86" y1="58.42" x2="22.86" y2="60.96" width="0.4064" layer="16"/>
 <wire x1="22.86" y1="60.96" x2="33.02" y2="60.96" width="0.4064" layer="16"/>
@@
 <wire x1="12.7" y1="20.32" x2="12.7" y2="15.24" width="0.4064" layer="16"/>
 <wire x1="63.5" y1="27.94" x2="66.04" y2="27.94" width="0.4064" layer="16"/>
+<contactref element="C4" pad="2"/>
+<contactref element="C5" pad="-"/>
+<wire x1="25.4" y1="22.86" x2="38.1" y2="22.86" width="0.4064" layer="16"/>
+<wire x1="38.1" y1="22.86" x2="45.72" y2="22.86" width="0.4064" layer="16"/>
+<wire x1="45.72" y1="22.86" x2="48.26" y2="22.86" width="0.4064" layer="16"/>
+<wire x1="45.72" y1="25.4" x2="45.72" y2="22.86" width="0.4064" layer="16"/>
 </signal>
 <signal name="N$1">
@@
 <contactref element="C4" pad="1"/>
 <wire x1="48.26" y1="25.4" x2="48.26" y2="27.94" width="0.4064" layer="16"/>
+<contactref element="C5" pad="+"/>
+<wire x1="38.1" y1="20.32" x2="43.18" y2="20.32" width="0.4064" layer="1"/>
+<wire x1="43.18" y1="20.32" x2="48.26" y2="25.4" width="0.4064" layer="1"/>
 </signal>
 <signal name="+3V3">
@@
 <wire x1="15.24" y1="10.16" x2="15.24" y2="12.7" width="0.4064" layer="16"/>
 </signal>
-<signal name="N$2">
-<contactref element="C4" pad="2"/>
-<contactref element="C5" pad="+"/>
-<wire x1="38.1" y1="20.32" x2="48.26" y2="20.32" width="0.4064" layer="16"/>
-<wire x1="48.26" y1="20.32" x2="48.26" y2="22.86" width="0.4064" layer="16"/>
-</signal>
 <signal name="LRCK">
